File: VERA-XE-HDMI-Expansion.kicad_pcb (KiCad board)
At the start: 4 copper layers, 89 x 37 mm, 67 parts, among them J1 CONN_HDMI_A, J2 CONN_SMD_HEADER_BOX_02x08_Odd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, U1 AMS1117-1.8, U2 MS9288C

Commit message: Autogenerated v1.1
Parts:
- moved R4 8.29 mm to (175.3, 90.6)
- moved R9 4.74 mm to (183.3, 94.2)
- moved LOGO2 3.73 mm to (172.7, 87.3)
- moved R11 1.40 mm to (189.5, 110.8)
- moved R3 1.40 mm to (175.5, 110.8)
- moved R5 1.40 mm to (170.5, 110.8)
- moved R6 1.40 mm to (185.5, 110.8)
Routing:
- net VGAGREEN: track 77.4 -> 88.3 mm, vias 2 -> 4
- net GND: track 151.4 -> 157.2 mm, vias 32 -> 33
- net VGABLUE: track 75.5 -> 78.6 mm
- net 5V: track 137.6 -> 135.1 mm
- net AUDIOL: track 20.6 -> 18.9 mm
- net AUDIOR: track 11.0 -> 12.3 mm
- net Net-(C26-Pad2): track 45.0 -> 43.7 mm
- net VGARED: track 63.3 -> 64.4 mm
