File: VERA-HDMI-Expansion.kicad_pcb (KiCad board)
At the start: 4 copper layers, 89 x 37 mm, 67 parts, among them J1 CONN_HDMI_A, J2 CONN_SMD_HEADER_BOX_02x08_Odd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, U1 AMS1117-1.8, U2 MS9288C

Commit message: 24.576Mhz Crystal Oscillator added
Parts:
- added C35: 22pF, Capacitor_SMD:C_0603_1608Metric_Pad1.08x0.95mm_HandSolder, F.Cu at (121.4, 89.5)
- added C36: 22pF, Capacitor_SMD:C_0603_1608Metric_Pad1.08x0.95mm_HandSolder, F.Cu at (121.4, 83.7)
- added Y1: 24.756Mhz, Crystal:Crystal_SMD_EuroQuartz_MT-4Pin_3.2x2.5mm, F.Cu at (121.4, 86.6)
Routing:
- net Net-(C36-Pad2): track 0.00 -> 16.8 mm, vias 0 -> 2
- net Net-(C35-Pad2): track 0.00 -> 16.8 mm, vias 0 -> 2
- net GND: track 157.2 -> 163.9 mm, vias 33 -> 35
