File: VERA-HDMI-Expansion.kicad_pcb (KiCad board)
At the start: 4 copper layers, 89 x 37 mm, 70 parts, among them J1 CONN_HDMI_A, J2 CONN_SMD_HEADER_BOX_02x08_Odd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, U1 AMS1117-1.8, U2 MS9288C, Y1 24.756Mhz

Commit message: Updated Crystal Oscillator Symbol from RetroBit Library
Parts:
- Y1: value 24.756Mhz -> 24.576Mhz
