File: VERA-HDMI-Expansion.sch (KiCad schematic (older format))
At the start: 67 parts, among them J1 CONN_HDMI_A, J2 CONN_SMD_HEADER_BOX_02x08_Odd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, U1 AMS1117-1.8, U2 MS9288C

Commit message: 24.576Mhz Crystal Oscillator added
Parts:
- added C35, C36: 22pF, Capacitor_SMD:C_0603_1608Metric_Pad1.08x0.95mm_HandSolder, symbol CCAP0603:22pF
- added Y1: 24.756Mhz, Crystal:Crystal_SMD_EuroQuartz_MT-4Pin_3.2x2.5mm, symbol RetroBitLab:24.756Mhz
Connections:
- wire segments 340 -> 354
Changed lines of the file:
@@
 Wire Wire Line
 	3370 7255 3695 7255
+$Comp
+L RetroBitLab:24.756Mhz Y1
+U 1 1 69040B10
+P 7980 6075
+F 0 "Y1" V 7865 5880 50  0000 L CNN
+F 1 "24.756Mhz" V 7725 5805 50  0000 L CNN
+F 2 "Crystal:Crystal_SMD_EuroQuartz_MT-4Pin_3.2x2.5mm" H 7580 6350 50  0001 C CNN
+F 3 "https://www.lcsc.com/datasheet/C9002.pdf" H 7980 6075 50  0001 C CNN
+F 4 "C41383247" H 7805 6450 50  0001 C CNN "LCSC"
+	1    7980 6075
+	0    1    1    0
+$EndComp
+$Comp
+L CCAP0603:22pF C35
+U 1 1 690661A6
+P 8250 5885
+F 0 "C35" V 8065 5885 50  0000 C CNN
+F 1 "22pF" V 8135 5900 50  0000 C CNN
+F 2 "Capacitor_SMD:C_0603_1608Metric_Pad1.08x0.95mm_HandSolder" H 8250 5885 50  0001 C CNN
+F 3 "https://lcsc.com/datasheet/lcsc_datasheet_2506131730_YAGEO-CC0603JRNPO9BN220_C105620.pdf" H 8250 5885 50  0001 C CNN
+F 4 "C105620" H 8250 5885 50  0001 C CNN "LCSC"
+	1    8250 5885
+	0    1    1    0
+$EndComp
+$Comp
+L CCAP0603:22pF C36
+U 1 1 69066D26
+P 8245 6255
+F 0 "C36" V 8130 6250 50  0000 C CNN
+F 1 "22pF" V 8295 6115 50  0000 C CNN
+F 2 "Capacitor_SMD:C_0603_1608Metric_Pad1.08x0.95mm_HandSolder" H 8245 6255 50  0001 C CNN
+F 3 "https://lcsc.com/datasheet/lcsc_datasheet_2506131730_YAGEO-CC0603JRNPO9BN220_C105620.pdf" H 8245 6255 50  0001 C CNN
+F 4 "C105620" H 8245 6255 50  0001 C CNN "LCSC"
+	1    8245 6255
+	0    1    1    0
+$EndComp
+Wire Wire Line
+	7980 5925 7980 5885
+Wire Wire Line
+	7980 5885 8150 5885
+Wire Wire Line
+	7980 6225 7980 6255
+Wire Wire Line
+	7980 6255 8145 6255
+Wire Wire Line
+	8180 6075 8495 6075
+Wire Wire Line
+	8495 6075 8495 5885
+Wire Wire Line
+	8495 5885 8350 5885
+Wire Wire Line
+	8345 6255 8495 6255
+Wire Wire Line
+	8495 6255 8495 6075
+Connection ~ 8495 6075
+$Comp
+L power:GND #PWR025
+U 1 1 690EB7CA
+P 8555 6075
+F 0 "#PWR025" H 8555 5825 50  0001 C CNN
+F 1 "GND" H 8560 5902 50  0000 C CNN
+F 2 "" H 8555 6075 50  0001 C CNN
+F 3 "" H 8555 6075 50  0001 C CNN
+	1    8555 6075
+	0    -1   -1   0
+$EndComp
+Wire Wire Line
+	8555 6075 8495 6075
+$Comp
+L power:GND #PWR024
+U 1 1 6914569A
+P 7780 6075
+F 0 "#PWR024" H 7780 5825 50  0001 C CNN
+F 1 "GND" H 7785 5902 50  0000 C CNN
+F 2 "" H 7780 6075 50  0001 C CNN
+F 3 "" H 7780 6075 50  0001 C CNN
+	1    7780 6075
+	0    1    1    0
+$EndComp
+Wire Wire Line
+	7980 5885 6745 5885
+Wire Wire Line
+	6745 5885 6745 5805
+Connection ~ 7980 5885
+Wire Wire Line
+	7980 6255 6620 6255
+Wire Wire Line
+	6620 6255 6620 5805
+Connection ~ 7980 6255
 $EndSCHEMATC
