File: VERA-HDMI-Expansion.sch (KiCad schematic (older format))
At the start: 70 parts, among them J1 CONN_HDMI_A, J2 CONN_SMD_HEADER_BOX_02x08_Odd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, U1 AMS1117-1.8, U2 MS9288C, Y1 24.756Mhz

Commit message: Updated Crystal Oscillator Symbol from RetroBit Library
Parts:
- removed Y1: 24.756Mhz, Crystal:Crystal_SMD_EuroQuartz_MT-4Pin_3.2x2.5mm, symbol RetroBitLab:24.756Mhz
- added Y1: 24.576Mhz, Crystal:Crystal_SMD_EuroQuartz_MT-4Pin_3.2x2.5mm, symbol RetroBitLab:24.576Mhz
Connections:
- wire segments 354 -> 355
Changed lines of the file:
@@
 Sheet 1 1
 Title "VERA HDMI Card"
-Date "2025-10-29"
+Date "2026-09-03"
 Rev "1.1"
 Comp "RetroBitLab"
@@
 L power:GND #PWR018
 U 1 1 6904AB93
-P 1865 5930
-F 0 "#PWR018" H 1865 5680 50  0001 C CNN
-F 1 "GND" H 1870 5757 50  0000 C CNN
-F 2 "" H 1865 5930 50  0001 C CNN
-F 3 "" H 1865 5930 50  0001 C CNN
-	1    1865 5930
+P 1865 5960
+F 0 "#PWR018" H 1865 5710 50  0001 C CNN
+F 1 "GND" H 2000 5890 50  0000 C CNN
+F 2 "" H 1865 5960 50  0001 C CNN
+F 3 "" H 1865 5960 50  0001 C CNN
+	1    1865 5960
 	1    0    0    -1
 $EndComp
@@
 Connection ~ 1865 5865
 Wire Wire Line
-	1865 5930 1865 5865
+	1865 5960 1865 5920
 $Comp
 L CCAP0805:22uF C33
@@
 	3370 7255 3695 7255
 $Comp
-L RetroBitLab:24.756Mhz Y1
-U 1 1 69040B10
-P 7980 6075
-F 0 "Y1" V 7865 5880 50  0000 L CNN
-F 1 "24.756Mhz" V 7725 5805 50  0000 L CNN
-F 2 "Crystal:Crystal_SMD_EuroQuartz_MT-4Pin_3.2x2.5mm" H 7580 6350 50  0001 C CNN
-F 3 "https://www.lcsc.com/datasheet/C9002.pdf" H 7980 6075 50  0001 C CNN
-F 4 "C41383247" H 7805 6450 50  0001 C CNN "LCSC"
-	1    7980 6075
-	0    1    1    0
-$EndComp
-$Comp
 L CCAP0603:22pF C35
 U 1 1 690661A6
@@
 	6620 6255 6620 5805
 Connection ~ 7980 6255
+$Comp
+L RetroBitLab:24.576Mhz Y1
+U 1 1 6A9ECC4E
+P 7980 6075
+F 0 "Y1" V 7860 5875 50  0000 L CNN
+F 1 "24.576Mhz" V 7735 5770 50  0000 L CNN
+F 2 "Crystal:Crystal_SMD_EuroQuartz_MT-4Pin_3.2x2.5mm" H 7580 6350 50  0001 C CNN
+F 3 "https://www.lcsc.com/datasheet/C9002.pdf" H 7980 6075 50  0001 C CNN
+F 4 "C41383247" H 7805 6450 50  0001 C CNN "LCSC"
+	1    7980 6075
+	0    1    1    0
+$EndComp
+$Comp
+L power:PWR_FLAG #FLG0101
+U 1 1 6A9F3FF2
+P 4265 5380
+F 0 "#FLG0101" H 4265 5455 50  0001 C CNN
+F 1 "PWR_FLAG" H 4275 5520 50  0000 C CNN
+F 2 "" H 4265 5380 50  0001 C CNN
+F 3 "~" H 4265 5380 50  0001 C CNN
+	1    4265 5380
+	1    0    0    -1
+$EndComp
+Connection ~ 4265 5380
+$Comp
+L power:PWR_FLAG #FLG0102
+U 1 1 6A9F568A
+P 10010 3080
+F 0 "#FLG0102" H 10010 3155 50  0001 C CNN
+F 1 "PWR_FLAG" H 10010 3253 50  0000 C CNN
+F 2 "" H 10010 3080 50  0001 C CNN
+F 3 "~" H 10010 3080 50  0001 C CNN
+	1    10010 3080
+	1    0    0    -1
+$EndComp
+Connection ~ 10010 3080
+$Comp
+L power:PWR_FLAG #FLG0103
+U 1 1 6AA13B81
+P 1865 5920
+F 0 "#FLG0103" H 1865 5995 50  0001 C CNN
+F 1 "PWR_FLAG" V 1765 6005 50  0000 L CNN
+F 2 "" H 1865 5920 50  0001 C CNN
+F 3 "~" H 1865 5920 50  0001 C CNN
+	1    1865 5920
+	0    -1   -1   0
+$EndComp
+Connection ~ 1865 5920
+Wire Wire Line
+	1865 5920 1865 5865
 $EndSCHEMATC
